Commit message: rbsherpa_xl_base.urdf.xacro: removed base-footprint's visual and erased a link name error

File: rbsherpa_description/urdf/bases/rbsherpa_xl_base.urdf.xacro (robot description, xacro)
@@ -10,10 +10,10 @@
     <xacro:if value="${publish_bf}">
       <link name="${prefix}base_footprint">
-        <visual>
+        <!--visual>
           <origin xyz="0 0 0" rpy="0 0 0" />
           <geometry>
             <box size="0.001 0.001 0.001" />
           </geometry>
-        </visual>
+        </visual-->
       </link>
       <joint name="${prefix}base_footprint_joint" type="fixed">
@@ -25,5 +25,5 @@
     </xacro:if>
     <!-- BASE_LINK -->
-    <link name="${prefix}base_link">   x:1.025 y:0.75 z:0.3
+    <link name="${prefix}base_link">
       <inertial>
         <mass value="25.0" />
